Commit message: left and right wheels axis aligned

File: urdf/mantaro.urdf (robot description, URDF)
Before this commit: robot mantaroboti 2, 8 links, 8 joints
Links:
- removed link caster_front_link
- removed link holder_link
- removed link plate_link
- added link caster_behind_link, mass 0.01; collision cylinder length=0.0176 radius=0.017; visual mesh filename=package://mantaro_description/meshes/caster_behind.stl
- link base_link: geometry visual mesh filename=package://mantaro_description/meshes/base.stl
- link wheel_left_link: geometry collision cylinder length=0.0206 radius=0.0352; visual mesh filename=package://mantaro_description/meshes/left_wheel.stl
- link wheel_right_link: geometry collision cylinder length=0.0206 radius=0.0350; visual mesh filename=package://mantaro_description/meshes/right_wheel.stl
Joints:
- removed joint caster_front_joint
- removed joint plate_to_holder_left
- removed joint plate_to_holder_right
- removed joint pole_to_plate
- added joint caster_behind_joint: type continuous, parent base_link, child caster_behind_link, origin xyz=-0.13 0 0.050 rpy=0 0 0, axis 0 1 0
- joint base_to_pole: origin xyz=0 0 .255 -> xyz=0 0 0.255
- joint wheel_left_joint: axis 1 0 0 -> 0 1 0; origin xyz=0 .07 0 rpy=0 0 0 -> xyz=0.1210 0.165 0.0551 rpy=0 0 0
- joint wheel_right_joint: origin xyz=0 -.16 0 rpy=0 0 0 -> xyz=0.10925 -0.16 0.0479 rpy=0 0 0

Commit message: merged with master

File: urdf/mantaro.urdf (robot description, URDF)
Before this commit: robot mantarobot, 6 links, 5 joints
Joints:
- joint caster_behind_joint: origin xyz=-0.13 0 0.050 rpy=0 0 0 -> xyz=-0.1286 0 0.04429 rpy=0 0 0

Commit message: pole axis aligned

File: urdf/mantaro.urdf (robot description, URDF)
Before this commit: robot mantarobot, 6 links, 5 joints
Joints:
- joint base_to_pole: axis (none) -> 0 0 1; type fixed -> continuous
